File: power.kicad_sch (KiCad schematic)
At the start: 24 parts, among them U10 TPS7A7001DDA, U8 TLV75733PDBVR

Commit message: Add more footprints!
Parts:
- C16, C17, C18, C19, C21, C22: footprint (none) -> Capacitor_SMD:C_0402_1005Metric_Pad0.74x0.62mm_HandSolder
- C23: footprint (none) -> Capacitor_THT:CP_Radial_D13.0mm_P5.00mm
- L2: footprint (none) -> Inductor_SMD:L_0603_1608Metric_Pad1.05x0.95mm_HandSolder
- R17, R20, R21, R22, R23, R40: footprint (none) -> Resistor_SMD:R_0402_1005Metric_Pad0.72x0.64mm_HandSolder

Commit message: More schematic work
Parts:
- D2, D3, D5: footprint (none) -> LED_SMD:LED_0603_1608Metric
Changed lines of the file:
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@@
 			)
 		)
-		(property "Footprint" ""
+		(property "Footprint" "LED_SMD:LED_0603_1608Metric"
 			(at 147.32 87.63 0)
 			(effects
@@
 			)
 		)
-		(property "Footprint" ""
+		(property "Footprint" "LED_SMD:LED_0603_1608Metric"
 			(at 177.8 87.63 0)
 			(effects
@@
 			)
 		)
-		(property "Footprint" ""
+		(property "Footprint" "LED_SMD:LED_0603_1608Metric"
 			(at 118.11 87.63 0)
 			(effects

Commit message: Power redesign
Parts:
- removed C18: 470uF, Capacitor_SMD:C_0402_1005Metric_Pad0.74x0.62mm_HandSolder, symbol Device:C_Polarized
- removed C19, C21: 10uF, Capacitor_SMD:C_0402_1005Metric_Pad0.74x0.62mm_HandSolder, symbol Device:C
- removed C22: 100nF, Capacitor_SMD:C_0402_1005Metric_Pad0.74x0.62mm_HandSolder, symbol Device:C
- removed C23: 3300uF, Capacitor_THT:CP_Radial_D13.0mm_P5.00mm, symbol Device:C_Polarized
- removed FB1: FerriteBead, symbol Device:FerriteBead
- removed L2: 15uH, Inductor_SMD:L_0603_1608Metric_Pad1.05x0.95mm_HandSolder, symbol Device:L
- removed R17: 50mR, Resistor_SMD:R_0402_1005Metric_Pad0.72x0.64mm_HandSolder, symbol Device:R
- removed R22: 221k, Resistor_SMD:R_0402_1005Metric_Pad0.72x0.64mm_HandSolder, symbol Device:R
- removed R23: 20k, Resistor_SMD:R_0402_1005Metric_Pad0.72x0.64mm_HandSolder, symbol Device:R
- removed U10: TPS7A7001DDA, Package_SO:TI_SO-PowerPAD-8, symbol Regulator_Linear:TPS7A7001DDA
- added C47: 10uF, symbol Device:C
- added C48, C49: 100nF, symbol Device:C
- added C50, C51: 47uF, symbol Device:C
- added C52: 75pF, symbol Device:C
- added C53: 1nF, symbol Device:C
- added D6: LED, LED_SMD:LED_0603_1608Metric, symbol Device:LED
- added FB2: FerriteBead, symbol Device:FerriteBead
- added L4: 10uH, symbol Device:L_Iron
- added R10: 100k, symbol Device:R
- added R11: 13.3k, symbol Device:R
- added R8: 1k, Resistor_SMD:R_0402_1005Metric_Pad0.72x0.64mm_HandSolder, symbol Device:R
- added TP5: TestPoint, TestPoint:TestPoint_Pad_D2.0mm, symbol Connector:TestPoint
- added U12: TPS54302, Package_TO_SOT_SMD:SOT-23-6, symbol Regulator_Switching:TPS54302
- R20, R21, R40: value 470R -> 1k
Connections:
- net +5V: now also FB2.2
- net GND: now also C47.2, C48.2, C50.2, C51.2, C53.2, R11.2, R8.2, U12.1 (GND)
- new net: C49.2, L4.1, U12.2 (SW)
- new net: C52.2, R10.2, R11.1, U12.4 (FB)
- new net: C53.1, U12.5 (EN)
- new net: C49.1, U12.6 (BOOT)
- new net: C50.1, C51.1, C52.1, FB2.1, L4.2, R10.1
- new net: D6.1 (K), R8.1
- new net +12V: C47.1, C48.1, D6.2 (A), TP5.1, U12.3 (VIN)
Other:
- note added: "Here's our power scheme: - VBUS is the input from the BEC (battery eliminator circuit) of the ESC. It's full of harmonics and is NOT clean at all. We use this to drive servos and NOTHING ELSE. - The 12V net is the battery raw input. This is used to power the rest of the flight computer - The 5V rail is generated by a TPS54302 switching supply from the 12V rail. - The 3.3V net is true 3.3v and is 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"
- note added: "There is an internal pullup here, so we don't need to connect EN (see datasheet)"
- note removed: "4.2V regulator"
- note removed: "5V Input filter from BEC"
- note removed: "APH0630T150M"
- note removed: "Cap omitted here because of previous caps"
- note removed: "Filter curve"
- note removed: "Here's our power scheme: - VBUS is the input from the BEC (battery eliminator circuit) of the ESC. It's full of harmonics and is NOT clean at all. We use this to drive servos and the rest of the power chain. - The 5V net is actually 4.2V. This is because the LDO is used as the final step in filtering the BEC, so there's a voltage drop. The only thing that is being fed by it is the 3.3V regulator,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"
- note removed: "Input bulk (pre-LC) Cin: 100-470 µF electrolytic Purpose: absorb ESC current spikes Voltage: ≥ 2× battery max ESR: not critical Main LC low-pass L1: 33 µH shielded power inductor DCR ≈ 0.27 Ω (good - provides damping) Current rating: ≥ 2× max rail current Saturation current: ≥ 2.5× load C1: 3300 µF electrolytic Voltage: ≥ 2× rail voltage ESR: 20-100 mΩ (perfect) 🧠 Results: Cutoff frequency ≈ 480 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"
- note removed: "LC Filter ~700Hz"
- note removed: "Low frequency filter cap"
- note removed: "R=0.04"
- note removed: "R=0.05"
- note removed: "R=0.113"
- note removed: "The purpose of this is to prevent ringing of the LC circuit, which can easily kill everything else"
- note removed: "Total system resistance ~0.2 ohms"
- moved on the sheet: C16, C17, U8

Commit message: Continue work
Parts:
- added J17: Screw_Terminal_01x02, lcsc:CONN-TH_2P-P5.00_WJ500V-5.08-2P, symbol Connector:Screw_Terminal_01x02
- C47, C48, C49, C50, C51, C52, C53: footprint (none) -> Capacitor_SMD:C_0402_1005Metric_Pad0.74x0.62mm_HandSolder
- R10, R11: footprint (none) -> Resistor_SMD:R_0402_1005Metric_Pad0.72x0.64mm_HandSolder
Connections:
- net +12V: now also J17.1 (Pin_1)
- net GND: now also J17.2 (Pin_2)
Other:
- note added: "C8465"

Commit message: Start PCB layout
Parts:
- FB2: footprint (none) -> Inductor_SMD:L_0805_2012Metric
- L4: footprint (none) -> lcsc:IND-SMD_L5.4-W5.2_MPCA-0518
Other:
- note added: "C5349679"
- note added: "C76818"
- note removed: "MPZ2012S221AT000"
Changed lines of the file:
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@@
 		(rev "V0")
 	)
-	(text "MPZ2012S221AT000\n"
-		(exclude_from_sim no)
-		(at 153.924 137.414 0)
+	(text "C76818"
+		(exclude_from_sim no)
+		(at 153.924 136.398 0)
 		(effects
 			(font
 				(size 0.508 0.508)
+				(thickness 0.1016)
+				(bold yes)
 			)
 		)
@@
 		)
 	)
+	(text "C5349679"
+		(exclude_from_sim no)
+		(at 100.33 136.144 0)
+		(effects
+			(font
+				(size 1.27 1.27)
+			)
+		)
+	)
 	(junction
 		(at 123.19 133.35)
@@
 			)
 		)
-		(property "Footprint" ""
+		(property "Footprint" "Inductor_SMD:L_0805_2012Metric"
 			(at 151.13 135.128 90)
 			(effects
@@
 			)
 		)
-		(property "Footprint" ""
+		(property "Footprint" "lcsc:IND-SMD_L5.4-W5.2_MPCA-0518"
 			(at 100.33 133.35 0)
 			(effects
