File: sensors.kicad_sch (KiCad schematic)
At the start: 37 parts, among them J10 Conn_Coaxial, U3 LSM6DSOXTR, U4 LIS3MDL, U5 BNO055, U6 BME280, U7 ATGM336H-5N31, Y3 32.768KHz 12.5pF

Commit message: Continue work
Parts:
- J10: footprint (none) -> lcsc:RF-SMD_FRF05002-JSS103M
- L1: footprint Inductor_SMD:L_0603_1608Metric_Pad1.05x0.95mm_HandSolder -> Inductor_SMD:L_0402_1005Metric_Pad0.77x0.64mm_HandSolder
Other:
- note added: "C88374"
Changed lines of the file:
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@@
 		)
 	)
+	(text "C88374"
+		(exclude_from_sim no)
+		(at 169.926 162.306 0)
+		(effects
+			(font
+				(size 1.27 1.27)
+			)
+		)
+	)
 	(junction
 		(at 35.56 143.51)
@@
 			)
 		)
-		(property "Footprint" "Inductor_SMD:L_0603_1608Metric_Pad1.05x0.95mm_HandSolder"
+		(property "Footprint" "Inductor_SMD:L_0402_1005Metric_Pad0.77x0.64mm_HandSolder"
 			(at 156.21 149.86 0)
 			(effects
@@
 			)
 		)
-		(property "Footprint" ""
+		(property "Footprint" "lcsc:RF-SMD_FRF05002-JSS103M"
 			(at 163.83 157.48 0)
 			(effects

Commit message: Start PCB layout
Parts:
- U7: footprint libsos41:GPSM-SMD_ATGM336H-TR -> lcsc:GPSM-SMD_ATGM336H-TR
Changed lines of the file:
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@@
 			)
 		)
-		(property "Footprint" "libsos41:GPSM-SMD_ATGM336H-TR"
+		(property "Footprint" "lcsc:GPSM-SMD_ATGM336H-TR"
 			(at 133.35 167.64 0)
 			(effects
