File: Zephyr.kicad_pcb (KiCad board)
At the start: 2 copper layers, 150 parts, among them J1 Conn_02x03_Counter_Clockwise, J10 Conn_Coaxial, J11 Conn_01x03, J12 Conn_01x07_Pin, J13 Conn_01x03, J14 Conn_01x06, J15 Micro_SD_Card, J16 Conn_Coaxial, J17 Screw_Terminal_01x02, J2 Conn_01x03, J3 Conn_01x03, J4 Conn_01x03, J5 Conn_01x03, J6 Conn_01x03, J7 Conn_01x03, J8 Conn_01x03, J9 Conn_01x03, Q1 MMBT3904, Q2 MMBT3904, SW4 SW_Push, U1 STM32F405RGT6, U11 E22-400M30S, U12 TPS54302, U2 PCA9685PW, U3 LSM6DSOXTR, U4 LIS3MDL, U5 BNO055, U6 BME280, U7 ATGM336H-5N31, U8 TLV75733PDBVR, U9 W25Q128JVS, Y1 32.768KHz 12.5pF, Y2 8MHz 12pF, Y3 32.768KHz 12.5pF

Commit message: Start layout
Parts:
- moved J17 192.3 mm to (66.5, 158.2)
- moved U12 190.4 mm to (57.8, 144.7), turned to 90 degrees
- moved R19 186.0 mm to (61.2, 110.1), turned to 90 degrees
- moved U7 185.1 mm to (70.0, 123.0), turned to -90 degrees
- moved L1 185.0 mm to (62.6, 120.3), turned to 90 degrees
- moved J10 178.2 mm to (60.0, 119.7), turned to 90 degrees
- moved R16 174.2 mm to (77.3, 123.0), turned to 180 degrees
- moved C47 173.2 mm to (68.5, 135.8)
- moved C48 173.2 mm to (68.5, 137.8)
- moved C49 173.2 mm to (68.5, 139.8)
- moved C50 173.2 mm to (68.5, 141.8)
- moved C51 173.2 mm to (68.5, 143.7)
- moved C52 173.2 mm to (68.5, 145.7)
- moved C53 173.2 mm to (68.5, 147.7)
- moved FB2 173.2 mm to (81.6, 150.7)
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Connections:
- J1 pad 1: /SYS_JTCK-SWCLK -> /SYS_JTMS-SWDIO
- J1 pad 2: /SYS_JTMS-SWDIO -> /SYS_JTCK-SWCLK
- U1 pad 62: unconnected-(U1-PB9-Pad62) -> /Guidance Sensors/BNO_RESET
Routing:
- net +3.3V: track 0.00 -> 3.55 mm
- net Net-(U1-VCAP_2): track 0.00 -> 1.84 mm
- net /RCC_OSC32_OUT: track 0.00 -> 0.69 mm
Other:
- board outline added: 110 x 60 mm
